File: KiCAD/Main/GPS/GPS.kicad_sch (KiCad schematic)
At the start: 28 parts, among them IC1 E22-900M22S, U1 MAX-M8Q, U2 PHA-23LN, U7 PHA-23LN

Commit message: Add files via upload
Parts:
- removed AE1, AE2: Antenna, symbol Device:Antenna
- removed C1, C13, C15, C16, C3, C6: 0.1u, symbol Device:C
- removed C12, C2: 0.001u, symbol Device:C
- removed C14, C5: 0.01u, symbol Device:C
- removed C17, C4: 1.2p, symbol Device:C
- removed IC1: E22-900M22S, E22-900M22S:E22-900M22S, symbol E22-900M22S:E22-900M22S
- removed JP1: SolderJumper_2_Open, symbol Jumper:SolderJumper_2_Open
- removed L1, L4: 1n, symbol Device:L
- removed L2, L3: 0.68u, symbol Device:L
- removed R1, R5: 1.21k, symbol Device:R
- removed R2: 10k, symbol Device:R
- removed R3, R4: 47, symbol Device:R
- removed U1: MAX-M8Q, RF_GPS:ublox_MAX, symbol RF_GPS:MAX-M8Q
- removed U2, U7: PHA-23LN, Package_TO_SOT_SMD:SOT-89-3, symbol RF_Amplifier:PHA-23LN

Commit message: Complete GPS section
Parts:
- added AE1: Antenna, symbol Device:Antenna
- added C1, C3, C6: 0.1u, symbol Device:C
- added C2: 0.001u, symbol Device:C
- added C4: 1.2p, symbol Device:C
- added C5: 0.01u, symbol Device:C
- added JP1: SolderJumper_2_Open, symbol Jumper:SolderJumper_2_Open
- added L1: 1n, symbol Device:L
- added L2: 0.68u, symbol Device:L
- added R1: 1.21k, symbol Device:R
- added R2: 10k, symbol Device:R
- added R3, R4: 47, symbol Device:R
- added U1: MAX-M8Q, RF_GPS:ublox_MAX, symbol RF_GPS:MAX-M8Q
- added U2: PHA-23LN, Package_TO_SOT_SMD:SOT-89-3, symbol RF_Amplifier:PHA-23LN
Connections:
- new net: R4.1, U1.2 (TXD)
- new net: AE1.1 (A), C4.1, L1.2
- new net: C3.1, L1.1
- new net: C1.2, C3.2, U2.1
- new net: C2.1, U1.11 (RF_IN)
- new net: R2.1, U1.13 (LNA_EN)
- new net: C5.2, C6.2, U1.14 (VCC_RF)
- new net: JP1.2 (B), U1.18 (~{SAFEBOOT})
- new net: R3.1, U1.3 (RXD)
- new net: C2.2, L2.2, R1.2, U2.3
- new net: C1.1, R1.1
- new net +3V3: JP1.1 (A), U1.6 (V_BCKP), U1.7 (VCC_IO), U1.8 (VCC)
- new net GND: C4.2, C5.1, C6.1, L2.1, R2.2, U1.1 (GND), U1.10 (GND), U1.12 (GND), U2.2 (GND)
- new net GPS RESET: U1.9 (~{RESET})
- new net GPS UART RX: R3.2
- new net GPS UART TX: R4.2
