File: KiCAD/Main/MCU.kicad_sch (KiCad schematic)
At the start: 8 parts, among them U1 STM32H730VBTx

Commit message: Add files via upload
Connections:
- net Camera RCC OSC32 IN is gone; now on net SD_MOSI: U1.8 (PC14)
- net Camera User BTN is gone; now on net SD_MISO: U1.7 (PC13)
- net SD_CLK: now also U1.80 (PC12); no longer U1.29 (PA5)
- net SD_MISO: no longer U1.90 (PB4(NJTRST))
- net SD_MOSI: no longer U1.31 (PA7)
- net SD_RESET: now reaches U1.79 (PC11)
- net BMP390 (SPI4) CS1: no longer names the net of U1.55 (PD8)
- net BMP390 (SPI4) CS2: no longer names the net of U1.56 (PD9)
- net BMP390 (SPI4) CS3: no longer names the net of U1.57 (PD10)
- net BNO085 CS: no longer names the net of U1.51 (PB12)
- net BNO085 MISO: no longer names the net of U1.53 (PB14)
- net BNO085 MOSI: no longer names the net of U1.54 (PB15)
- net BNO085 SCK: no longer names the net of U1.52 (PB13)
- net Camera (I2C1) SCL: no longer names the net of U1.95 (PB8)
- net Camera (I2C1) SDA: no longer names the net of U1.96 (PB9)
- net Camera DCMI D0: no longer names the net of U1.63 (PC6)
- net Camera DCMI D1: no longer names the net of U1.64 (PC7)
- net Camera DCMI D2: no longer names the net of U1.65 (PC8)
- net Camera DCMI D3: no longer names the net of U1.66 (PC9)
- net Camera DCMI D4: no longer names the net of U1.3 (PE4)
- net Camera DCMI D5: no longer names the net of U1.84 (PD3)
- net Camera DCMI D6: no longer names the net of U1.4 (PE5)
- net Camera DCMI D7: no longer names the net of U1.5 (PE6)
- net Camera DCMI HSYNC: no longer names the net of U1.28 (PA4)
- net Camera DCMI VSYNC: no longer names the net of U1.93 (PB7)
- net Camera Debug SWCLK: no longer names the net of U1.76 (PA14(JTCK)
- net Camera Debug SWDIO: no longer names the net of U1.72 (PA13(JTMS)
- net Camera PWDN: no longer names the net of U1.61 (PD14)
- net Camera RCC MCO1: no longer names the net of U1.67 (PA8)
- net Camera RCC OSC IN: no longer names the net of U1.12 (PH0)
- net Camera RCC OSC OUT: no longer names the net of U1.13 (PH1)
- net Camera RCC OSC32 OUT: no longer names the net of U1.9 (PC15)
- net Camera RX: no longer names the net of U1.37 (PE7)
- net Camera Reset: no longer names the net of U1.62 (PD15)
- net Camera TX: no longer names the net of U1.38 (PE8)
- net GPS_RESET: no longer names the net of U1.24 (PA2)
- net GPS_RX renamed USER_BTN
- net GPS_TX renamed USER_LED
- net SD_CS: no longer names the net of U1.77 (PA15(JTDI))
- net SHT41 (SPI4) CS1: no longer names the net of U1.39 (PE9)
- net SHT41 (SPI4) CS2: no longer names the net of U1.40 (PE10)
- net SHT41 (SPI4) CS3: no longer names the net of U1.41 (PE11)
- net SHT41 and BMP390 (SPI4) MISO: no longer names the net of U1.43 (PE13)
- net SHT41 and BMP390 (SPI4) MOSI: no longer names the net of U1.44 (PE14)
- net SHT41 and BMP390 (SPI4) SCK: no longer names the net of U1.42 (PE12)
- net Thermistor 1: no longer names the net of U1.15 (PC0)
- net Thermistor 2: no longer names the net of U1.16 (PC1)
- net Thermistor 3: no longer names the net of U1.17 (PC2_C)
- net Thermistor 4: no longer names the net of U1.18 (PC3_C)
- net USER BTN: no longer names the net of U1.34 (PB0)
- net USER LED: no longer names the net of U1.33 (PC5)
