File: KiCAD/Main/Power_Essentials.kicad_sch (KiCad schematic)
At the start: 26 parts, among them J1 USB_C_Receptacle_USB2.0_16P, J2 Micro_SD_Card_Det2, J4 Screw_Terminal_01x09, J5 Screw_Terminal_01x09, SW1 RESET, SW2 USER, U2 LM2596S-3.3, U3 LM2596S-5, U4 TPS2121RUXR

Commit message: Add files via upload
Changed lines of the file:
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@@
 		)
 	)
-	(hierarchical_label "5V_STABILIZED"
+	(global_label "3V3_STABILIZED"
 		(shape input)
-		(at 191.77 39.37 180)
+		(at 130.81 153.67 180)
+		(fields_autoplaced yes)
 		(effects
 			(font
@@
 			)
 			(justify right)
+		)
+		(property "Intersheetrefs" "${INTERSHEET_REFS}"
+			(at 112.9477 153.67 0)
+			(effects
+				(font
+					(size 1.27 1.27)
+				)
+				(justify right)
+				(hide yes)
+			)
+		)
+	)
+	(global_label "5V_STABILIZED"
+		(shape input)
+		(at 191.77 39.37 180)
+		(fields_autoplaced yes)
+		(effects
+			(font
+				(size 1.27 1.27)
+			)
+			(justify right)
+		)
+		(property "Intersheetrefs" "${INTERSHEET_REFS}"
+			(at 175.1172 39.37 0)
+			(effects
+				(font
+					(size 1.27 1.27)
+				)
+				(justify right)
+				(hide yes)
+			)
 		)
 	)
@@
 		)
 	)
-	(hierarchical_label "3V3_STABILIZED"
-		(shape input)
-		(at 130.81 153.67 180)
-		(effects
-			(font
-				(size 1.27 1.27)
-			)
-			(justify right)
-		)
-	)
