File: KiCAD/Main/Main.kicad_sch (KiCad schematic)
At the start: 2 parts, among them J7 Conn_02x05_Top_Bottom_Mountin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

Commit message: Update RF sys and footprints
Parts:
- J7: footprint (none) -> Connector_IDC:IDC-Header_2x05_P2.54mm_Horizontal
Changed lines of the file:
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@@
 			)
 		)
-		(property "Footprint" ""
+		(property "Footprint" "Connector_IDC:IDC-Header_2x05_P2.54mm_Horizontal"
 			(at 53.34 95.25 0)
 			(effects
