File: KiCAD/Main/Main.kicad_pcb (KiCad board)
At the start: 2 copper layers, 5 parts, among them U1 STM32H730VBTx, U2 LM2596S-3.3, U3 LM2596S-5

Commit message: Add files via upload
Parts:
- added <Designator>?: E22-900T22S, E22-900T22S:E22-900T22S, F.Cu at (131.3, 94.0)

Commit message: Submit design for review
Parts:
- removed the U1 at (121.3, 65.0)
- added D1: Green 5mA, LED_SMD:LED_0603_1608Metric, F.Cu at (61.5, 80.4)
- added D3: 1N5820, Diode_THT:D_DO-201AD_P15.24mm_Horizontal, F.Cu at (43.3, 87.1)
- added D4: 1N5820, Diode_THT:D_DO-201AD_P15.24mm_Horizontal, F.Cu at (43.3, 93.8)
- added D5: 1N5820, Diode_THT:D_DO-201AD_P15.24mm_Horizontal, F.Cu at (43.3, 100.6)
- added Q1: AO3400A, Package_TO_SOT_SMD:SOT-23, F.Cu at (63.4, 86.1)
- added Q2: AO3400A, Package_TO_SOT_SMD:SOT-23, F.Cu at (63.4, 90.7)
- added Q3: AO3400A, Package_TO_SOT_SMD:SOT-23, F.Cu at (63.4, 95.3)
- added R1: 10K, Resistor_SMD:R_0603_1608Metric, F.Cu at (61.4, 72.8)
- added R2: 100K, Resistor_SMD:R_0603_1608Metric, F.Cu at (61.4, 75.3)
- added R4: 634, Resistor_SMD:R_0603_1608Metric, F.Cu at (61.4, 77.9)
- added SW1: RESET, Button_Switch_SMD:SW_Push_1P1T_NO_Vertical_Wuerth_434133025816, F.Cu at (62.8, 64.5)
- added SW2: USER, Button_Switch_SMD:SW_Push_1P1T_NO_Vertical_Wuerth_434133025816, F.Cu at (62.8, 69.2)
- added U17: SHT4x, Sensor_Humidity:Sensirion_DFN-4_1.5x1.5mm_P0.8mm_SHT4x_NoCentralPad, F.Cu at (76.4, 63.6)
- added U4: STM32H750VBTx, Package_QFP:LQFP-100_14x14mm_P0.5mm, F.Cu at (48.5, 68.0)
- added U5: MAX-M8Q, RF_GPS:ublox_MAX, F.Cu at (74.2, 89.6)
- added U6: PHA-23LN, Package_TO_SOT_SMD:SOT-89-3, F.Cu at (71.2, 98.5)
- added U9: BME280, Package_LGA:Bosch_LGA-8_2.5x2.5mm_P0.65mm_ClockwisePinNumbering, F.Cu at (70.5, 64.3)
- renumbered D1 to D2, U2 to U1
Connections:
- D2 pad 1: Net-(D1-K) -> Net-(D2-K)
- U1 pad 1: Net-(U2-VIN) -> Net-(U1-VIN)
- U1 pad 2: Net-(D1-K) -> Net-(D2-K)
- U1 pad 3: Net-(U2-GND) -> GND
- U1 pad 5: Net-(U2-GND) -> GND

Commit message: Update RF sys and footprints
Parts:
- added BZ1: Buzzer, Buzzer_Beeper:MagneticBuzzer_PUI_SMT-1028-T-2-R, F.Cu at (246.7, 72.1)
- added C1: 680u, Capacitor_SMD:C_0603_1608Metric, F.Cu at (216.6, 41.9)
- added C10: 100n, Capacitor_SMD:C_0603_1608Metric, F.Cu at (234.0, 70.1)
- added C11: 100n, Capacitor_SMD:C_0603_1608Metric, F.Cu at (234.0, 72.6)
- added C12: 100n, Capacitor_SMD:C_0603_1608Metric, F.Cu at (234.0, 75.1)
- added C13: 1u, Capacitor_SMD:C_0603_1608Metric, F.Cu at (234.0, 77.6)
- added C14: 4.7u, Capacitor_SMD:C_0603_1608Metric, F.Cu at (234.0, 80.1)
- added C15: 220u, Capacitor_SMD:C_0603_1608Metric, F.Cu at (216.6, 47.0)
- added C2: 10n, Capacitor_SMD:C_0603_1608Metric, F.Cu at (216.6, 44.4)
- added C21: 100n, Capacitor_SMD:C_0603_1608Metric, F.Cu at (257.4, 67.5)
- added C22: 100n, Capacitor_SMD:C_0603_1608Metric, F.Cu at (257.4, 70.1)
- added C23: 2.2u, Capacitor_SMD:C_0603_1608Metric, F.Cu at (257.4, 72.6)
- added C24: 100n, Capacitor_SMD:C_0603_1608Metric, F.Cu at (257.4, 75.1)
- added C25: 100n, Capacitor_SMD:C_0603_1608Metric, F.Cu at (257.4, 77.6)
- added C26: 100n, Capacitor_SMD:C_0603_1608Metric, F.Cu at (250.9, 46.9)
- added C27: 100n, Capacitor_SMD:C_0603_1608Metric, F.Cu at (250.9, 49.4)
- added C28: 100n, Capacitor_SMD:C_0603_1608Metric, F.Cu at (250.9, 51.9)
- added C29: 100n, Capacitor_SMD:C_0603_1608Metric, F.Cu at (263.6, 42.9)
- added C3: 2.2u, Capacitor_SMD:C_0603_1608Metric, F.Cu at (230.0, 67.5)
- added C30: 100n, Capacitor_SMD:C_0603_1608Metric, F.Cu at (263.6, 45.4)
- added C31: 100n, Capacitor_SMD:C_0603_1608Metric, F.Cu at (263.6, 47.9)
- added C32: 100n, Capacitor_SMD:C_0603_1608Metric, F.Cu at (263.6, 50.4)
- added C33: 100n, Capacitor_SMD:C_0603_1608Metric, F.Cu at (263.6, 52.9)
- added C34: 100n, Capacitor_SMD:C_0603_1608Metric, F.Cu at (263.6, 55.4)
- added C35: 100n, Capacitor_SMD:C_0603_1608Metric, F.Cu at (268.6, 67.5)
- added C36: 0.1u, Capacitor_SMD:C_0603_1608Metric, F.Cu at (238.0, 67.5)
- added C4: 2.2u, Capacitor_SMD:C_0603_1608Metric, F.Cu at (230.0, 70.1)
- added C5: 100N, Capacitor_SMD:C_0603_1608Metric, F.Cu at (230.0, 72.6)
- added C6: 1u, Capacitor_SMD:C_0603_1608Metric, F.Cu at (230.0, 75.1)
- added C7: 100n, Capacitor_SMD:C_0603_1608Metric, F.Cu at (230.0, 77.6)
- added C8: 100n, Capacitor_SMD:C_0603_1608Metric, F.Cu at (230.0, 80.1)
- added C9: 100n, Capacitor_SMD:C_0603_1608Metric, F.Cu at (234.0, 67.5)
- added D6: MBRS340, Diode_SMD:D_SMC, F.Cu at (220.6, 70.2)
- added D7: MBRS340, Diode_SMD:D_SMC, F.Cu at (232.1, 44.5)
- added J1: Micro_SD_Card_Det2, Connector_Card:microSD_HC_Hirose_DM3AT-SF-PEJM5, F.Cu at (206.2, 50.0)
- added J2: Screw_Terminal_01x09, Connector_Phoenix_MSTB:PhoenixContact_MSTBVA_2,5_9-G_1x09_P5.00mm_Vertical, F.Cu at (202.4, 24.8)
- added J3: Screw_Terminal_01x09, Connector_Phoenix_MSTB:PhoenixContact_MSTBVA_2,5_9-G_1x09_P5.00mm_Vertical, F.Cu at (202.4, 35.9)
- added J4: USB_C_Receptacle_USB2.0_16P, Connector_USB:USB_C_Receptacle_HRO_TYPE-C-31-M-12, F.Cu at (220.5, 56.5)
- added J7: Conn_02x05_Top_Bottom_MountingPin, Connector_IDC:IDC-Header_2x05_P2.54mm_Horizontal, F.Cu at (200.8, 72.4)
- added J8: Conn_Coaxial, Connector_Coaxial:U.FL_Molex_MCRF_73412-0110_Vertical, F.Cu at (256.0, 58.3)
- added JP2: BMI270 TMR Toggle, Resistor_SMD:R_0603_1608Metric_Pad0.98x0.95mm_HandSolder, F.Cu at (267.8, 55.0)
- added JP3: BMP390 TMR Toggle, Resistor_SMD:R_0603_1608Metric_Pad0.98x0.95mm_HandSolder, F.Cu at (255.1, 46.9)
- added L1: 33u, Inductor_SMD:L_0603_1608Metric, F.Cu at (216.6, 49.5)
- added Q4: 2N7002, Package_TO_SOT_SMD:SOT-23, F.Cu at (247.7, 80.2)
- added R10: 47, Resistor_SMD:R_0603_1608Metric, F.Cu at (250.9, 56.5)
- added R11: 47, Resistor_SMD:R_0603_1608Metric, F.Cu at (250.9, 59.0)
- added R12: 100, Resistor_SMD:R_0603_1608Metric, F.Cu at (238.0, 72.6)
- added R14: 10k, Resistor_SMD:R_0603_1608Metric, F.Cu at (257.4, 80.1)
- added R15: 10k, Resistor_SMD:R_0603_1608Metric, F.Cu at (257.4, 82.6)
- added R17: 10k, Resistor_SMD:R_0603_1608Metric, F.Cu at (268.6, 70.1)
- added R18: 10k, Resistor_SMD:R_0603_1608Metric, F.Cu at (268.6, 72.6)
- added R19: 10k, Resistor_SMD:R_0603_1608Metric, F.Cu at (224.7, 44.4)
- added R20: 10k, Resistor_SMD:R_0603_1608Metric, F.Cu at (224.7, 47.0)
- added R21: 10k, Resistor_SMD:R_0603_1608Metric, F.Cu at (224.7, 49.5)
- added R28: 30, Resistor_SMD:R_0603_1608Metric, F.Cu at (250.9, 61.5)
- added R29: 1k, Resistor_SMD:R_0603_1608Metric, F.Cu at (238.0, 75.1)
- added R3: 100k, Resistor_SMD:R_0603_1608Metric, F.Cu at (220.7, 41.9)
- added R5: 100k, Resistor_SMD:R_0603_1608Metric, F.Cu at (220.7, 44.4)
- added R6: 10, Resistor_SMD:R_0603_1608Metric, F.Cu at (220.7, 47.0)
- added R7: 5.1k, Resistor_SMD:R_0603_1608Metric, F.Cu at (220.7, 49.5)
- added R8: 5.1k, Resistor_SMD:R_0603_1608Metric, F.Cu at (224.7, 41.9)
- added R9: 10k, Resistor_SMD:R_0603_1608Metric, F.Cu at (238.0, 70.1)
- added U10: ~, E22-900M22S:E22-900M22S, F.Cu at (257.4, 29.0)
- added U11: BMP390L, BMP390L:XDCR_BMP390L, F.Cu at (250.7, 43.9)
- added U12: BMP390L, BMP390L:XDCR_BMP390L, F.Cu at (254.3, 43.9)
- added U13: BMP390L, BMP390L:XDCR_BMP390L, F.Cu at (257.8, 43.9)
- added U14: BMI270, BMI270:XDCR_BMI270, F.Cu at (268.3, 43.6)
- added U15: BMI270, BMI270:XDCR_BMI270, F.Cu at (268.3, 47.7)
- added U16: BMI270, BMI270:XDCR_BMI270, F.Cu at (268.3, 51.7)
- added U2: TPS2121RUXR, TPS2121RUXR:IC_TPS2121RUXR, F.Cu at (240.1, 42.9)
- added U3: BMM350, BMM350:BGA9C40P3X3_128X128X50, F.Cu at (261.3, 71.7)
- added U7: ISM6HG256x, ISM6HG256XTR:U_LGA-14L_2p5X3p0X0p83_STM, F.Cu at (262.2, 68.4)
- added Y2: SiT8008xx-2x-xxE (25MHz), Oscillator:Oscillator_SMD_SiT_PQFN-4Pin_3.2x2.5mm, F.Cu at (242.6, 80.2)
- moved <Designator>? 149.0 mm to (272.0, 143.0)
- moved D1 149.0 mm to (202.2, 129.4)
- moved D2 149.0 mm to (233.1, 108.1)
- moved D2 149.0 mm to (233.1, 114.9)
- moved D3 149.0 mm to (184.0, 136.1)
- moved D4 149.0 mm to (184.0, 142.8)
- moved D5 149.0 mm to (184.0, 149.6)
- moved Q1 149.0 mm to (204.1, 135.1)
- moved Q2 149.0 mm to (204.1, 139.7)
- moved Q3 149.0 mm to (204.1, 144.4)
- moved R1 149.0 mm to (202.1, 121.9)
- moved R2 149.0 mm to (202.1, 124.4)
- moved R4 149.0 mm to (202.1, 126.9)
- moved SW1 149.0 mm to (203.5, 113.5)
- moved SW2 149.0 mm to (203.5, 118.2)
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Connections:
- net /Microcontroller/~{RESET} renamed /~{RESET}
- U4 pad 12: unconnected-(U4-PH0-Pad12) -> /Microcontroller/~{OSC_OUT}
- U4 pad 66: /IMUs/BNO_RST -> unconnected-(U4-PC9-Pad66)

Commit message: Begin PCB layout
Parts:
- removed R28: 30, Resistor_SMD:R_0603_1608Metric
- removed the U3 at (241.5, 136.8)
- removed U6: PHA-23LN, Package_TO_SOT_SMD:SOT-89-3
- moved U14 214.6 mm to (74.0, 134.7)
- moved C29 213.2 mm to (72.7, 137.9)
- moved <Designator>? 208.4 mm to (83.0, 55.4), turned to 180 degrees
- moved C31 208.3 mm to (75.7, 137.9), turned to 180 degrees
- moved U11 206.0 mm to (74.0, 149.7)
- moved C30 205.6 mm to (80.0, 137.9)
- moved JP3 205.0 mm to (81.3, 155.6), turned to 180 degrees
- moved U16 204.6 mm to (81.2, 134.6)
- moved C26 203.0 mm to (74.0, 146.3), turned to 180 degrees
- moved U12 202.8 mm to (81.2, 149.7)
- moved C32 200.7 mm to (83.0, 137.9), turned to 180 degrees
- moved JP2 200.2 mm to (81.1, 127.4)
- moved U15 199.7 mm to (88.5, 134.7)
- moved U13 199.7 mm to (88.5, 149.7)
- moved R21 199.3 mm to (65.2, 169.0), turned to -90 degrees
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Connections:
- U5 pad 13: Net-(U5-LNA_EN) -> +3V3
- U5 pad 14: +3V3 -> Net-(U5-VCC_RF)
Routing:
- net (no net): track 0.00 -> 12.1 mm, vias 0 -> 2
- net GND: track 0.00 -> 6.01 mm, vias 0 -> 1
Other:
- copper layers 2 -> 4

Commit message: 30%
Parts:
- removed <Designator>?: E22-900T22S, E22-900T22S:E22-900T22S
- added C16: 10n, Capacitor_SMD:C_0603_1608Metric, F.Cu at (108.0, 42.5)
- added J9: Conn_Coaxial, Connector_Coaxial:U.FL_Molex_MCRF_73412-0110_Vertical, F.Cu at (74.3, 45.5)
- added L2: 47n, Inductor_SMD:L_0603_1608Metric, F.Cu at (111.3, 43.2)
- added R13: 10, Resistor_SMD:R_0603_1608Metric, F.Cu at (108.0, 44.2)
- U10: footprint E22-900M22S:E22-900M22S -> E22-900T22S:E22-900T22S
- moved R1 48.6 mm to (76.6, 88.5)
- moved R2 48.6 mm to (80.2, 88.5)
- moved SW2 47.3 mm to (86.5, 80.8)
- moved SW1 45.8 mm to (78.5, 80.8)
- moved J7 41.5 mm to (96.7, 77.8), turned to 90 degrees
- moved J4 35.4 mm to (128.2, 69.8)
- moved R21 35.0 mm to (95.3, 151.2), turned to 180 degrees
- moved Q3 32.7 mm to (91.2, 152.1), turned to -90 degrees
- moved D5 29.5 mm to (109.2, 158.1), turned to -90 degrees
- moved R20 28.3 mm to (95.3, 156.1), turned to 180 degrees
- moved U10 27.2 mm to (91.1, 51.0), turned to -90 degrees
- moved J8 26.4 mm to (116.8, 43.2), turned to -90 degrees
- moved U5 26.2 mm to (115.0, 52.2)
- moved Q2 25.8 mm to (91.2, 157.0), turned to -90 degrees
- moved R10 25.5 mm to (108.0, 52.4)
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Connections:
- C10 pad 1: Net-(U4-VDDA) -> +3V3
- C10 pad 2: +3V3 -> GND
- C11 pad 1: Net-(U4-VDDA) -> +3V3
- C11 pad 2: +3V3 -> GND
- C12 pad 1: Net-(U4-VDDA) -> +3V3
- C12 pad 2: +3V3 -> GND
- C13 pad 1: Net-(U4-VDDA) -> +3V3
- C13 pad 2: +3V3 -> GND
- C14 pad 1: Net-(U4-VDDA) -> +3V3
- C14 pad 2: +3V3 -> GND
- C6 pad 1: +3V3 -> GND
- C7 pad 1: Net-(U4-VDDA) -> +3V3
- C7 pad 2: +3V3 -> GND
- C8 pad 1: Net-(U4-VDDA) -> +3V3
- C8 pad 2: +3V3 -> GND
- C9 pad 1: Net-(U4-VDDA) -> +3V3
- C9 pad 2: +3V3 -> GND
- U10 pad 1: /RF/NOTE: Using built-in coaxial antenna port -> Net-(J9-In)
- U4 pad 100: Net-(U4-VDDA) -> +3V3
- U4 pad 11: Net-(U4-VDDA) -> +3V3
- U4 pad 21: Net-(U4-VDDA) -> +3V3
- U4 pad 27: Net-(U4-VDDA) -> +3V3
- U4 pad 50: Net-(U4-VDDA) -> +3V3
- U4 pad 75: Net-(U4-VDDA) -> +3V3
Routing:
- net GND: track 6.01 -> 154.1 mm, vias 1 -> 14
- net /Microcontroller/SD_Det: track 0.00 -> 77.2 mm
- net +3V3: track 0.00 -> 60.7 mm, vias 0 -> 7
- net Net-(U1-VIN): track 0.00 -> 59.7 mm
- net /~{RESET}: track 0.00 -> 53.5 mm
- net Net-(D2-K): track 0.00 -> 52.2 mm
- net /Microcontroller/USER_BTN: track 0.00 -> 39.3 mm
- net Net-(J4-CC1): track 0.00 -> 36.1 mm
- net Net-(D6-A): track 0.00 -> 32.2 mm
- net Net-(D5-K): track 0.00 -> 31.3 mm
- net Net-(D7-A): track 0.00 -> 29.0 mm
- net Net-(J4-CC2): track 0.00 -> 27.4 mm
- net Net-(U4-PC13): track 0.00 -> 26.6 mm
- net Net-(D4-K): track 0.00 -> 24.3 mm
- net Net-(D3-K): track 0.00 -> 17.3 mm
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Other:
- board outline added: 80.2 x 150 mm
